Commit message: modified auto move, add teleop files for the new model

File: turtlebot3_description/urdf/turtlebot3_burger.urdf.xacro (robot description, xacro)
@@ -7,5 +7,5 @@
     <parent link="base_footprint"/>
     <child link="base_link"/>
-    <origin xyz="3.5 2.0 0.010" rpy="0 0 0"/>
+    <origin xyz="0.3 0.3 0.10" rpy="0 0 0"/>
   </joint>
   <link name="base_link">
